File: design_files_32U4/project V0.kicad_pcb (KiCad board)
At the start: 2 copper layers, 25.4 x 25.4 mm, 27 parts, among them CON1 AVR-ISP-6, J2 Conn_01x06, J4 Conn_01x08, SW1 RESET, U1 ATMEGA32U4-AU, U2 MIC5225-3.3, X3 USB_OTG, Y1 8 Mhz

Commit message: Updates
Other:
- board text added: "+ ISP -"
- board text removed: "- ISP +"
Changed lines of the file:
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@@
     (links 77)
     (no_connects 0)
-    (area 142.164999 86.284999 167.715001 111.835001)
+    (area 125.73 78.580001 182.145715 114.300001)
     (thickness 1.6)
     (drawings 19)
@@
     (visible_elements 7FFEFFFF)
     (pcbplotparams
-      (layerselection 0x00030_80000001)
+      (layerselection 0x010f0_80000001)
       (usegerberextensions false)
       (excludeedgelayer true)
@@
       (outputformat 1)
       (mirror false)
-      (drillshape 1)
+      (drillshape 0)
       (scaleselection 1)
-      (outputdirectory ""))
+      (outputdirectory gerbers/))
   )
   (net 0 "")
@@
     (arrow2b (pts (xy 167.64 81.280001) (xy 166.513496 81.866422)))
   )
-  (gr_text "- ISP +" (at 156.845 94.234) (layer B.SilkS)
+  (gr_text "+ ISP -" (at 156.845 94.234) (layer B.SilkS)
     (effects (font (size 1.25 1.25) (thickness 0.3)) (justify mirror))
   )
