File: design_files_32U4/project.sch (KiCad schematic (older format))
At the start: 25 parts, among them CON1 AVR-ISP-6, J2 Beetja Bottom, J4 Beetja Top, SW1 RESET, U1 ATMEGA32U4-AU, U2 MIC5225-3.3, X3 USB_OTG, Y1 8 Mhz

Commit message: Updates
Parts:
- J2: value Beetja Bottom -> Beetje Bottom
- J4: value Beetja Top -> Beetje Top
Other:
- note added: "Beetje Footprint"
- note removed: "Beetja Footprint"
Changed lines of the file:
@@
 P 3000 5450
 F 0 "J4" H 3000 5850 50  0000 C CNN
-F 1 "Beetja Top" H 3000 4950 50  0000 C CNN
+F 1 "Beetje Top" H 3000 4950 50  0000 C CNN
 F 2 "footprints:Pin_Header_Straight_1x08_Pitch2.54mm" H 3000 5450 50  0001 C CNN
 F 3 "" H 3000 5450 50  0001 C CNN
@@
 P 3650 5350
 F 0 "J2" H 3650 5650 50  0000 C CNN
-F 1 "Beetja Bottom" H 3650 4950 50  0000 C CNN
+F 1 "Beetje Bottom" H 3650 4950 50  0000 C CNN
 F 2 "footprints:Pin_Header_Straight_1x06_Pitch2.54mm" H 3650 5350 50  0001 C CNN
 F 3 "" H 3650 5350 50  0001 C CNN
@@
 	4250 4900 2200 4900
 Text Notes 2250 5000 0    60   ~ 0
-Beetja Footprint
+Beetje Footprint
 $EndSCHEMATC
